File: docs/4-digit/v1/4-digit-v1.kicad_sch (KiCad schematic)
At the start: 47 parts, among them P1 (UART on the board), P2 (NMEA / NTP device), Q1 8550, Q2 8550, Q3 8550, Q4 8550, Q5 8550, Q6 8550, Q7 8550, SW1 SW_PUSH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

Commit message: Updated documentation
Parts:
- removed DS5, DS6: 7SEGMENTS, symbol stc_diyclock-rescue:7SEGMENTS
- removed Q5, Q6: 8550, TO-92, symbol stc_diyclock-rescue:S8550
- removed R18, R19: 10k, symbol stc_diyclock-rescue:R
- renumbered SW1 to S1, SW2 to S2
Connections:
- net   : now also U2.7 (P1.4/ADC4)
- net A5: no longer names the net of U2.21 (~{INT2}/P3.6)
- net A5: now also P2.2 (Pin_2)
- net A6: no longer names the net of U2.22 (~{INT3}/P3.7)
- net Rx renamed Rx, S2
- net Rx, S2: now also S2.2; no longer P2.2 (Pin_2)
- removed net S2: S2.2, U2.7 (P1.4/ADC4)
Other:
- note added: "4 digit DIY clock with NMEA hardware switch"
- note added: "December 2024"
- note removed: "6 digit DIY clock with NMEA hardware switch"
- note removed: "November 2024"
- moved on the sheet: C1, D1, DS1, DS2, DS3, DS4, P1, P2, Q1, Q2, Q3, Q4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
